Commit message: added robot functionality to the world plugin

File: src/kinect_v2/urdf/kinect_v2.urdf.xacro (robot description, xacro)
@@ -2,9 +2,9 @@
 <robot name="kinect_v2" xmlns:xacro="http://ros.org/wiki/xacro">
 <xacro:include filename="$(find kinect_v2)/urdf/kinect_v2.gazebo.xacro" />
-    <property name="M_PI" value="3.14159" />
+    <xacro:property name="M_PI" value="3.14159" />
     <!-- Kinect2 and mount assembly -->
     <xacro:macro name="kinect_v2" params=" parent *origin">
         <joint name="kinect2_joint" type="fixed">
-            <insert_block name="origin" />
+            <xacro:insert_block name="origin" />
             <parent link="${parent}" />
             <child link="kinect2_base_link" />
