Commit message: added classify option

File: src/jackal_velodyne/urdf/VLP-16.urdf.xacro (robot description, xacro)
@@ -2,5 +2,5 @@
 <robot xmlns:xacro="http://www.ros.org/wiki/xacro" name="VLP-16">
   <xacro:property name="M_PI" value="3.1415926535897931" />
-  <xacro:macro name="VLP-16" params="*origin parent:=base_link name:=velodyne topic:=/velodyne_points hz:=10 lasers:=16 samples:=1875 collision_range:=0.3 min_range:=0.9 max_range:=130.0 noise:=0.008 min_angle:=-${M_PI} max_angle:=${M_PI} gpu:=false">
+  <xacro:macro name="VLP-16" params="*origin parent:=base_link name:=velodyne topic:=/velodyne_points hz:=10 lasers:=16 samples:=1875 collision_range:=0.3 min_range:=0.9 max_range:=130.0 noise:=0.008 min_angle:=-${M_PI} max_angle:=${M_PI} gpu:=false classify:=true">
     <joint name="${name}_base_mount_joint" type="fixed">
       <xacro:insert_block name="origin" />
@@ -84,13 +84,25 @@
             </noise>
           </ray>
-          <plugin name="gazebo_ros_laser_controller" filename="libcustom_velodyne_gpu.so">
-            <topicName>${topic}</topicName>
-            <frameName>${name}</frameName>
-            <min_range>${min_range}</min_range>
-            <max_range>${max_range}</max_range>
-            <gaussianNoise>${noise}</gaussianNoise>
-            <robot_name>jackal</robot_name>
-            <building_name>building</building_name>
-          </plugin>
+          <xacro:if value="${classify}">
+            <plugin name="gazebo_ros_laser_controller" filename="libcustom_velodyne_gpu.so">
+                <topicName>${topic}</topicName>
+                <frameName>${name}</frameName>
+                <min_range>${min_range}</min_range>
+                <max_range>${max_range}</max_range>
+                <gaussianNoise>${noise}</gaussianNoise>
+                <robot_name>jackal</robot_name>
+                <building_name>building</building_name>
+                <classify>true</classify>
+            </plugin>
+          </xacro:if>
+          <xacro:unless value="${classify}">
+            <plugin name="gazebo_ros_laser_controller" filename="libgazebo_ros_velodyne_gpu_laser.so">
+                <topicName>${topic}</topicName>
+                <frameName>${name}</frameName>
+                <min_range>${min_range}</min_range>
+                <max_range>${max_range}</max_range>
+                <gaussianNoise>${noise}</gaussianNoise>
+            </plugin>
+          </xacro:unless>
         </sensor>
       </xacro:if>
@@ -126,13 +138,25 @@
             </noise>
           </ray>
-          <plugin name="gazebo_ros_laser_controller" filename="libcustom_velodyne.so">
-            <topicName>${topic}</topicName>
-            <frameName>${name}</frameName>
-            <min_range>${min_range}</min_range>
-            <max_range>${max_range}</max_range>
-            <gaussianNoise>${noise}</gaussianNoise>
-            <robot_name>jackal</robot_name>
-            <building_name>building</building_name>
-          </plugin>
+        <xacro:if value="${classify}">
+            <plugin name="gazebo_ros_laser_controller" filename="libcustom_velodyne.so">
+                <topicName>${topic}</topicName>
+                <frameName>${name}</frameName>
+                <min_range>${min_range}</min_range>
+                <max_range>${max_range}</max_range>
+                <gaussianNoise>${noise}</gaussianNoise>
+                <robot_name>jackal</robot_name>
+                <building_name>building</building_name>
+                <classify>true</classify>
+            </plugin>
+          </xacro:if>
+          <xacro:unless value="${classify}">
+            <plugin name="gazebo_ros_laser_controller" filename="libgazebo_ros_velodyne_laser.so">
+                <topicName>${topic}</topicName>
+                <frameName>${name}</frameName>
+                <min_range>${min_range}</min_range>
+                <max_range>${max_range}</max_range>
+                <gaussianNoise>${noise}</gaussianNoise>
+            </plugin>
+          </xacro:unless>
         </sensor>
       </xacro:unless>

File: src/jackal_velodyne/urdf/jackal_velodyne.urdf.xacro (robot description, xacro)
@@ -308,8 +308,16 @@
 	</gazebo>
   <!-- VLP-16 -->
-  <xacro:include filename="$(find jackal_velodyne)/urdf/VLP-16.urdf.xacro"/>
-  <VLP-16 parent="support_link3" name="velodyne" topic="/velodyne_points" hz="10" samples="1024" gpu="true" lasers="33" max_range="30">
-    <origin xyz="0 0 0" rpy="0 0 0" />
-  </VLP-16>
+  <xacro:if value="$(optenv CLASSIFY 1)">
+    <xacro:include filename="$(find jackal_velodyne)/urdf/VLP-16.urdf.xacro"/>
+    <VLP-16 parent="support_link3" name="velodyne" topic="/velodyne_points" hz="10" samples="1024" gpu="true" lasers="33" max_range="30" classify="true">
+        <origin xyz="0 0 0" rpy="0 0 0" />
+    </VLP-16>
+  </xacro:if>
+  <xacro:unless value="$(optenv CLASSIFY 1)">
+    <xacro:include filename="$(find jackal_velodyne)/urdf/VLP-16.urdf.xacro"/>
+    <VLP-16 parent="support_link3" name="velodyne" topic="/velodyne_points" hz="10" samples="1024" gpu="true" lasers="33" max_range="30" classify="false">
+        <origin xyz="0 0 0" rpy="0 0 0" />
+    </VLP-16>
+  </xacro:unless>
   <!--xacro:include filename="$(find jackal_velodyne)/urdf/VLP-16.urdf.xacro"/>
   <VLP-16 parent="support_link3" name="no_gpu_velodyne" topic="/no_gpu_points" hz="10" samples="1024" gpu="false" lasers="33" max_range="30">
