Commit message: trying to get custom camera plgin to work

File: src/jackal_velodyne/urdf/viewbot.urdf.xacro (robot description, xacro)
@@ -1,5 +1,5 @@
 <?xml version="1.0"?>
 <robot name="viewbot_link" xmlns:xacro="http://ros.org/wiki/xacro">
-<xacro:include filename="$(find jackal_velodyne)/urdf/viewbot.gazebo.xacro" />
+<!--xacro:include filename="$(find jackal_velodyne)/urdf/viewbot.gazebo.xacro" /-->
     <xacro:property name="M_PI" value="3.14159" />
     <xacro:macro name="viewbot_link" params=" filepath name parent *origin">
@@ -11,5 +11,44 @@
         <link name="${name}_base_link"/>
         <!-- gazebo extensions -->
-        <xacro:viewbot filepath="${filepath}" link_name="${name}_base_link" topic_name="${name}"/>
+        <!--xacro:viewbot filepath="${filepath}" link_name="${name}_base_link" topic_name="${name}"/-->
+        <gazebo reference="${name}_base_link">
+            <sensor name="viewbot" type="camera">
+                <camera>
+                    <!--save enabled="true">
+                        <path>${filepath}${name}</path>
+                    </save-->
+                    <horizontal_fov>1.047</horizontal_fov>
+                    <image>
+                        <width>1920</width>
+                        <height>1080</height>
+                    </image>
+                    <clip>
+                        <near>0.1</near>
+                        <far>100</far>
+                    </clip>
+                </camera>
+                <plugin name="${name}_controller" filename="libcustom_camera.so">
+                    <alwaysOn>true</alwaysOn>
+                    <updateRate>0.0</updateRate>
+                    <cameraName>${name}</cameraName>
+                    <imageTopicName>image_raw</imageTopicName>
+                    <cameraInfoTopicName>camera_info</cameraInfoTopicName>
+                    <frameName>${name}_base_link</frameName>
+                    <hackBaseline>0.0</hackBaseline>
+                    <distortionK1>0.0</distortionK1>
+                    <distortionK2>0.0</distortionK2>
+                    <distortionK3>0.0</distortionK3>
+                    <distortionT1>0.0</distortionT1>
+                    <distortionT2>0.0</distortionT2>
+                    <CxPrime>0</CxPrime>
+                    <Cx>0.0</Cx>
+                    <Cy>0.0</Cy>
+                    <focalLength>0.0</focalLength>
+                </plugin>
+                <always_on>1</always_on>
+                <update_rate>30</update_rate>
+            </sensor>
+        <material value="Gazebo/Red" />
+      </gazebo>
     </xacro:macro>
 </robot>
