Commit message: added stationary actor detection to post-classifier

File: src/jackal_velodyne/urdf/jackal_velodyne.urdf.xacro (robot description, xacro)
@@ -312,4 +312,8 @@
     <origin xyz="0 0 0" rpy="0 0 0" />
   </VLP-16>
+  <!--xacro:include filename="$(find jackal_velodyne)/urdf/VLP-16.urdf.xacro"/>
+  <VLP-16 parent="support_link3" name="no_gpu_velodyne" topic="/no_gpu_points" hz="10" samples="1024" gpu="false" lasers="33" max_range="30">
+    <origin xyz="0 0 0" rpy="0 0 0" />
+  </VLP-16-->
   <xacro:include filename="$(find kinect_v2)/urdf/kinect_v2.urdf.xacro" />
     <xacro:kinect_v2  parent="support_link3">

Commit message: Added first and third person views

File: src/jackal_velodyne/urdf/jackal_velodyne.urdf.xacro (robot description, xacro)
@@ -329,4 +329,18 @@
                 rpy="0 0 0" />
    </xacro:kinect_v2>
+   <!--xacro:include filename="$(find jackal_velodyne)/urdf/first_person.urdf.xacro" /-->
+  <xacro:include filename="$(find jackal_velodyne)/urdf/viewbot.urdf.xacro" />
+    <xacro:viewbot_link  name="first_person" parent="support_link3">
+        <origin xyz="0 0 0"
+                rpy="0 0 0" />
+    </xacro:viewbot_link>
+    <xacro:viewbot_link  name="third_person_rear" parent="base_link">
+        <origin xyz="-4 0 1"
+                rpy="0 0.2 0" />
+    </xacro:viewbot_link>
+    <xacro:viewbot_link  name="third_person" parent="base_link">
+        <origin xyz="4 0 1"
+                rpy="0 0.2 3.14" />
+    </xacro:viewbot_link>
 <!-- default samples = 1024 -->
   <!-- VHDL-32E -->

Commit message: Added FPV views that are automatically converted to mp4 files

File: src/jackal_velodyne/urdf/jackal_velodyne.urdf.xacro (robot description, xacro)
@@ -1,4 +1,6 @@
 <?xml version="1.0"?>
 <robot name="jackal" xmlns:xacro="http://www.ros.org/wiki/xacro">
+  <xacro:arg name="filepath" default = "/tmp" />
+  <xacro:property name="filepath" value = "$(arg filepath)" />
   <xacro:property name="PI" value="3.1415926535897931" />
   <xacro:property name="wheelbase" value="0.262" />
@@ -330,14 +332,14 @@
    </xacro:kinect_v2>
    <!--xacro:include filename="$(find jackal_velodyne)/urdf/first_person.urdf.xacro" /-->
-  <xacro:include filename="$(find jackal_velodyne)/urdf/viewbot.urdf.xacro" />
-    <xacro:viewbot_link  name="first_person" parent="support_link3">
+  <xacro:include  filename="$(find jackal_velodyne)/urdf/viewbot.urdf.xacro" />
+    <xacro:viewbot_link filepath="${filepath}" name="first_person" parent="support_link3">
         <origin xyz="0 0 0"
                 rpy="0 0 0" />
     </xacro:viewbot_link>
-    <xacro:viewbot_link  name="third_person_rear" parent="base_link">
+    <xacro:viewbot_link filepath="${filepath}" name="third_person_rear" parent="base_link">
         <origin xyz="-4 0 1"
                 rpy="0 0.2 0" />
     </xacro:viewbot_link>
-    <xacro:viewbot_link  name="third_person" parent="base_link">
+    <xacro:viewbot_link  filepath="${filepath}" name="third_person" parent="base_link">
         <origin xyz="4 0 1"
                 rpy="0 0.2 3.14" />

File: src/jackal_velodyne/urdf/viewbot.gazebo.xacro (robot description, xacro)
@@ -4,8 +4,11 @@
   <material>Gazebo/Grey</material>
   </gazebo>
-<xacro:macro name="viewbot" params="link_name topic_name">
+<xacro:macro name="viewbot" params="filepath link_name topic_name">
   <gazebo reference="${link_name}">
         <sensor name="viewbot" type="camera">
             <camera>
+                <save enabled="true">
+                    <path>${filepath}${topic_name}</path>
+                </save>
                 <horizontal_fov>1.047</horizontal_fov>
                 <image>
@@ -20,22 +23,4 @@
             <always_on>1</always_on>
             <update_rate>30</update_rate>
-            <plugin name = "camera_controller" filename = "libgazebo_ros_camera.so">
-                <alwaysOn>true</alwaysOn>
-                <updateRate>0.0</updateRate>
-                <cameraName>${topic_name}</cameraName>
-                <imageTopicName>image_raw</imageTopicName>
-                <cameraInfoTopicName>camera_info</cameraInfoTopicName>
-                <frameName>${link_name}</frameName>
-                <hackBaseline>0.0</hackBaseline>
-                <distortionK1>0.0</distortionK1>
-                <distortionK2>0.0</distortionK2>
-                <distortionK3>0.0</distortionK3>
-                <distortionT1>0.0</distortionT1>
-                <distortionT2>0.0</distortionT2>
-                <CxPrime>0</CxPrime>
-                <Cx>0.0</Cx>
-                <Cy>0.0</Cy>
-                <focalLength>0.0</focalLength>
-            </plugin>
         </sensor>
     <material value="Gazebo/Red" />
@@ -43,2 +28,20 @@
 </xacro:macro>
 </robot>
+<!--plugin name = "camera_controller" filename = "libgazebo_ros_camera.so">
+    <alwaysOn>true</alwaysOn>
+    <updateRate>0.0</updateRate>
+    <cameraName>${topic_name}</cameraName>
+    <imageTopicName>image_raw</imageTopicName>
+    <cameraInfoTopicName>camera_info</cameraInfoTopicName>
+    <frameName>${link_name}</frameName>
+    <hackBaseline>0.0</hackBaseline>
+    <distortionK1>0.0</distortionK1>
+    <distortionK2>0.0</distortionK2>
+    <distortionK3>0.0</distortionK3>
+    <distortionT1>0.0</distortionT1>
+    <distortionT2>0.0</distortionT2>
+    <CxPrime>0</CxPrime>
+    <Cx>0.0</Cx>
+    <Cy>0.0</Cy>
+    <focalLength>0.0</focalLength>
+</plugin-->

File: src/jackal_velodyne/urdf/viewbot.urdf.xacro (robot description, xacro)
@@ -3,5 +3,5 @@
 <xacro:include filename="$(find jackal_velodyne)/urdf/viewbot.gazebo.xacro" />
     <xacro:property name="M_PI" value="3.14159" />
-    <xacro:macro name="viewbot_link" params=" name parent *origin">
+    <xacro:macro name="viewbot_link" params=" filepath name parent *origin">
         <joint name="${name}_joint" type="fixed">
             <xacro:insert_block name="origin" />
@@ -11,5 +11,5 @@
         <link name="${name}_base_link"/>
         <!-- gazebo extensions -->
-        <xacro:viewbot link_name="${name}_base_link" topic_name="${name}"/>
+        <xacro:viewbot filepath="${filepath}" link_name="${name}_base_link" topic_name="${name}"/>
     </xacro:macro>
 </robot>

Commit message: improved exiting from master.sh

File: src/jackal_velodyne/urdf/jackal_velodyne.urdf.xacro (robot description, xacro)
@@ -322,8 +322,4 @@
     </VLP-16>
   </xacro:unless>
-  <!--xacro:include filename="$(find jackal_velodyne)/urdf/VLP-16.urdf.xacro"/>
-  <VLP-16 parent="support_link3" name="no_gpu_velodyne" topic="/no_gpu_points" hz="10" samples="1024" gpu="false" lasers="33" max_range="30">
-    <origin xyz="0 0 0" rpy="0 0 0" />
-  </VLP-16-->
   <xacro:include filename="$(find kinect_v2)/urdf/kinect_v2.urdf.xacro" />
     <xacro:kinect_v2  parent="support_link3">
@@ -331,6 +327,5 @@
                 rpy="0 0 0" />
    </xacro:kinect_v2>
-   <!--xacro:include filename="$(find jackal_velodyne)/urdf/first_person.urdf.xacro" /-->
-  <xacro:include  filename="$(find jackal_velodyne)/urdf/viewbot.urdf.xacro" />
+   <xacro:include  filename="$(find jackal_velodyne)/urdf/viewbot.urdf.xacro" />
     <xacro:viewbot_link filepath="${filepath}" name="first_person" parent="support_link3">
         <origin xyz="0 0 0"
@@ -338,11 +333,16 @@
     </xacro:viewbot_link>
     <xacro:viewbot_link filepath="${filepath}" name="third_person_rear" parent="base_link">
-        <origin xyz="-4 0 1"
-                rpy="0 0.2 0" />
+        <origin xyz="-6 0 2"
+                rpy="0 0.3 0" />
     </xacro:viewbot_link>
     <xacro:viewbot_link  filepath="${filepath}" name="third_person" parent="base_link">
-        <origin xyz="4 0 1"
+        <origin xyz="6 0 2"
                 rpy="0 0.2 3.14" />
     </xacro:viewbot_link>
+</robot>
+  <!--xacro:include filename="$(find jackal_velodyne)/urdf/VLP-16.urdf.xacro"/>
+  <VLP-16 parent="support_link3" name="no_gpu_velodyne" topic="/no_gpu_points" hz="10" samples="1024" gpu="false" lasers="33" max_range="30">
+    <origin xyz="0 0 0" rpy="0 0 0" />
+  </VLP-16-->
 <!-- default samples = 1024 -->
   <!-- VHDL-32E -->
@@ -351,3 +351,2 @@
     <origin xyz="0 0 0.6" rpy="0 0 0" />
   </HDL-32E> -->
-</robot>

Commit message: testing two-parter

File: src/jackal_velodyne/urdf/jackal_velodyne.urdf.xacro (robot description, xacro)
@@ -1,6 +1,6 @@
 <?xml version="1.0"?>
 <robot name="jackal" xmlns:xacro="http://www.ros.org/wiki/xacro">
-  <xacro:arg name="filepath" default = "/tmp" />
-  <xacro:property name="filepath" value = "$(arg filepath)" />
+  <!--xacro:arg name="filepath" default = "/tmp" /-->
+  <!--xacro:property name="filepath" value = "$(arg filepath)" /-->
   <xacro:property name="PI" value="3.1415926535897931" />
   <xacro:property name="wheelbase" value="0.262" />

Commit message: Big cleanup

File: src/jackal_velodyne/urdf/jackal_velodyne.urdf.xacro (robot description, xacro)
@@ -225,13 +225,4 @@
   <!-- Bring in simulation data for Gazebo. -->
   <xacro:include filename="$(find jackal_description)/urdf/jackal.gazebo" />
-  <!-- Optional standard accessories, including their simulation data. The rendering
-       of these into the final description is controlled by optenv variables, which
-       default each one to off.-->
-  <xacro:include filename="$(find jackal_velodyne)/urdf/accessories.urdf.xacro" />
-  <!-- Optional custom includes. -->
-  <xacro:if value="$(optenv JACKAL_URDF_EXTRAS 0)">
-    <xacro:include filename="$(env JACKAL_URDF_EXTRAS)" />
-  </xacro:if>
-<!-- tests below -->
   <!-- added support -->
   <link name="support_link1">
@@ -328,25 +319,2 @@
    </xacro:kinect_v2>
 </robot>
-   <!--xacro:include  filename="$(find jackal_velodyne)/urdf/viewbot.urdf.xacro" />
-    <xacro:viewbot_link filepath="${filepath}" name="first_person" parent="support_link3">
-        <origin xyz="0 0 0"
-                rpy="0 0 0" />
-    </xacro:viewbot_link>
-    <xacro:viewbot_link filepath="${filepath}" name="third_person_rear" parent="base_link">
-        <origin xyz="-6 0 2"
-                rpy="0 0.3 0" />
-    </xacro:viewbot_link>
-    <xacro:viewbot_link  filepath="${filepath}" name="third_person" parent="base_link">
-        <origin xyz="6 0 2"
-                rpy="0 0.2 3.14" />
-    </xacro:viewbot_link-->
-  <!--xacro:include filename="$(find jackal_velodyne)/urdf/VLP-16.urdf.xacro"/>
-  <VLP-16 parent="support_link3" name="no_gpu_velodyne" topic="/no_gpu_points" hz="10" samples="1024" gpu="false" lasers="33" max_range="30">
-    <origin xyz="0 0 0" rpy="0 0 0" />
-  </VLP-16-->
-<!-- default samples = 1024 -->
-  <!-- VHDL-32E -->
-<!--   <xacro:include filename="$(find velodyne_description)/urdf/HDL-32E.urdf.xacro"/>
-  <HDL-32E parent="base_link" name="velodyne_2" topic="/velodyne_points_2" hz="10" samples="1024" gpu="false">
-    <origin xyz="0 0 0.6" rpy="0 0 0" />
-  </HDL-32E> -->
